Commit message: urdf

File: werdna_description/urdf/consts.xacro (robot description, xacro)
@@ -27,8 +27,6 @@
     <xacro:property name="wheel_radius" value="0.06"/>
     <xacro:property name="wheel_length" value="0.02"/>
-    <xacro:property name="motor_radius" value="0.04"/>
-    <xacro:property name="motor_thickness" value="0.035"/>
-    <xacro:property name="gearbox_radius" value="0.04"/>
-    <xacro:property name="gearbox_thickness" value="0.042"/>
+    <xacro:property name="gearbox_radius" value="0.055"/>
+    <xacro:property name="gearbox_thickness" value="0.0738"/>
     <xacro:property name="imu_length" value="0.01"/>
     <xacro:property name="imu_width" value="0.01"/>
@@ -37,13 +35,8 @@
     <xacro:property name="rod_width" value="0.02"/>
     <xacro:property name="rod_height" value="0.148"/>
-    <xacro:property name="knee_rod_length" value="0.035"/>
-    <xacro:property name="knee_rod_width" value="0.02"/>
-    <xacro:property name="knee_rod_height" value="0.148"/>
     <!-- Masses -->
-    <xacro:property name="chassis_mass" value="1.5"/>
+    <xacro:property name="chassis_mass" value="2.0"/>
     <xacro:property name="rod_mass" value="0.1"/>
-    <xacro:property name="knee_rod_mass" value="0.1"/>
     <xacro:property name="wheel_mass" value="0.5"/>
-    <xacro:property name="motor_mass" value="0.3"/>
     <xacro:property name="gearbox_mass" value="0.3"/>
     <xacro:property name="imu_mass" value="0.001"/>
@@ -54,11 +47,8 @@
     <xacro:property name="imu_offset_x" value="0"/>
     <xacro:property name="imu_offset_y" value="0"/>
-    <xacro:property name="imu_offset_z" value="${chassis_height/2 + imu_height/2}"/>
+    <xacro:property name="imu_offset_z" value="0"/>
     <xacro:property name="gearbox_offset_x" value="0"/>
     <xacro:property name="gearbox_offset_y" value="${chassis_width/2 + gearbox_thickness/2}"/>
     <xacro:property name="gearbox_offset_z" value="0"/>
-    <xacro:property name="motor_offset_x" value="${-rod_height}"/>
-    <xacro:property name="motor_offset_y" value="0"/>
-    <xacro:property name="motor_offset_z" value="${motor_thickness/2 + rod_length/2}"/>
     <xacro:property name="hip_offset_x" value="${-rod_height}"/>
     <xacro:property name="hip_offset_y" value="0"/>

File: werdna_description/urdf/werdna.xacro (robot description, xacro)
@@ -3,5 +3,4 @@
     <xacro:include filename="consts.xacro"/>
     <xacro:include filename='inertial_macros.xacro'/>
-    <!-- Base Link -->
     <!-- Chassis -->
     <link name="base_link">
@@ -25,29 +24,11 @@
     </link>
     <!-- imu -->
-    <link name="imu_link">
-        <xacro:inertial_box mass="${imu_mass}" x="${imu_length}" y="${imu_width}" z="${imu_height}">
-            <origin xyz="0 0 0" rpy="0 0 0"/>
-        </xacro:inertial_box>
-        <visual>
-            <origin xyz="0.0 0.0 0.0" rpy="0.0 0.0 0.0"/>
-            <geometry>
-                <box size="${imu_length} ${imu_width} ${imu_height}"/>
-            </geometry>
-            <material name="white"/>
-        </visual>
-        <collision>
-            <origin xyz="0.0 0.0 0.0" rpy="0.0 0.0 0.0"/>
-            <geometry>
-                <box size="${imu_length} ${imu_width} ${imu_height}"/>
-            </geometry>
-            <material name="white"/>
-        </collision>
-    </link>
+    <!-- <link name="imu_link"></link> -->
     <!-- imu joint -->
-    <joint name="imu_joint" type="fixed">
+    <!-- <joint name="imu_joint" type="fixed">
         <origin xyz="${imu_offset_x} ${imu_offset_y} ${imu_offset_z}" rpy="0.0 0.0 0.0"/>
         <parent link="base_link"/>
         <child link="imu_link"/>
-    </joint>
+    </joint> -->
     <!-- Left Hip - Gearbox -->
     <link name="left_hip_motor_link">
@@ -71,5 +52,5 @@
     </link>
     <joint name="left_hip_motor_joint" type="revolute">
-        <origin xyz="0.0 ${gearbox_offset_y} 0.0" rpy="${pi/2} -0.524 0.0"/>
+        <origin xyz="0.0 ${gearbox_offset_y} 0.0" rpy="${pi/2} -${pi/6} 0.0"/>
         <parent link="base_link"/>
         <child link="left_hip_motor_link"/>
@@ -77,117 +58,63 @@
         <limit lower="${low_limit}" upper="${high_limit}" velocity="${velocity}" effort="${effort}"/>
     </joint>
-    <!-- Left Hip - Hip -->
     <link name="left_hip_link">
         <visual>
-            <origin xyz="-${rod_height/2} 0 0" rpy="0 ${pi/2} 0"/>
-            <geometry>
-                <box size="${rod_length} ${rod_width} ${rod_height}"/>
-            </geometry>
-            <material name="red"/>
-        </visual>
-        <collision>
-            <origin xyz="-${rod_height/2} 0 0" rpy="0 ${pi/2} 0"/>
-            <geometry>
-                <box size="${rod_length} ${rod_width} ${rod_height}"/>
-            </geometry>
-            <material name="red"/>
-        </collision>
-        <xacro:inertial_box mass="${rod_mass}" x="${rod_length}" y="${rod_width}" z="${rod_height}">
-            <origin xyz="-${rod_height/2} 0 0" rpy="0 ${pi/2} 0"/>
+             <origin xyz="-${rod_height/2} 0 0" rpy="0 ${pi/2} 0"/>
+            <geometry>
+                <box size="${rod_length} ${rod_width} ${rod_height}" rpy="0 0 0"/>
+            </geometry>
+            <material name="red"/>
+        </visual>
+        <collision>
+             <origin xyz="-${rod_height/2} 0 0" rpy="0 ${pi/2} 0"/>
+            <geometry>
+                <box size="${rod_length} ${rod_width} ${rod_height}" rpy="0 0 0"/>
+            </geometry>
+            <material name="red"/>
+        </collision>
+        <xacro:inertial_box mass="${rod_mass}" x="${rod_length}" y="${rod_width}" z="${rod_height}">
+             <origin xyz="-${rod_height/2} 0 0" rpy="0 ${pi/2} 0"/>
         </xacro:inertial_box>
     </link>
     <joint name="left_hip_joint" type="fixed">
-        <origin xyz="0.0 0.0 -${hip_offset_z}" rpy="0.0 0.0 0.0"/>
+        <origin xyz="0.0 0 -${gearbox_thickness/2 + rod_length/2}" rpy="0 0 0"/>
         <parent link="left_hip_motor_link"/>
         <child link="left_hip_link"/>
     </joint>
-    <!-- Left Knee - Motor -->
-    <link name="left_knee_motor_link">
-        <visual>
-            <origin xyz="${rod_height} 0 0" rpy="0 0 0"/>
-            <geometry>
-                <cylinder radius="${motor_radius}" length="${motor_thickness}"/>
-            </geometry>
-            <material name="red"/>
-        </visual>
-        <collision>
-            <origin xyz="${rod_height} 0 0" rpy="0 0 0"/>
-            <geometry>
-                <cylinder radius="${motor_radius}" length="${motor_thickness}"/>
-            </geometry>
-            <material name="red"/>
-        </collision>
-        <xacro:inertial_cylinder mass="${motor_mass}" length="${motor_thickness}" radius="${motor_radius}">
-            <origin xyz="${rod_height} 0 0" rpy="0 0 0"/>
-        </xacro:inertial_cylinder>
-    </link>
-    <joint name="left_knee_motor_joint" type="fixed">
-        <origin xyz="${motor_offset_x} 0 -${motor_offset_z}" rpy="0.0 0 0"/>
+    <link name="left_knee_link">
+        <visual>
+             <origin xyz="0 0 ${rod_height/2}" rpy="0.0 0 ${pi/2}"/>
+            <geometry>
+                <box size="${rod_length} ${rod_width} ${rod_height}" rpy="0 0 0"/>
+            </geometry>
+            <material name="red"/>
+        </visual>
+        <collision>
+             <origin xyz="0 0 ${rod_height/2}" rpy="0 0 ${pi/2}"/>
+            <geometry>
+                <box size="${rod_length} ${rod_width} ${rod_height}" rpy="0 0 0"/>
+            </geometry>
+            <material name="red"/>
+        </collision>
+        <xacro:inertial_box mass="${rod_mass}" x="${rod_length}" y="${rod_width}" z="${rod_height}">
+             <origin xyz="0 0 ${rod_height/2}" rpy="0 0 ${pi/2}"/>
+        </xacro:inertial_box>
+    </link>
+    <joint name="left_knee_joint" type="revolute">
+        <origin xyz="-${rod_height} 0 0" rpy="${pi/2} 0 ${pi/6}"/>
         <parent link="left_hip_link"/>
-        <child link="left_knee_motor_link"/>
-    </joint>
-    <!-- Left Hip - Link Outer-->
-    <link name="left_knee_outer_link">
-        <visual>
-            <origin xyz="0 0 ${rod_height/2}" rpy="0 0 0"/>
-            <geometry>
-                <box size="${rod_length} ${rod_width} ${rod_height}"/>
-            </geometry>
-            <material name="red"/>
-        </visual>
-        <collision>
-            <origin xyz="0 0 ${rod_height/2}" rpy="0 0 0"/>
-            <geometry>
-                <box size="${rod_length} ${rod_width} ${rod_height}"/>
-            </geometry>
-            <material name="red"/>
-        </collision>
-        <xacro:inertial_box mass="${rod_mass}" x="${rod_length}" y="${rod_width}" z="${rod_height}">
-            <origin xyz="0 0 ${rod_height/2}" rpy="0 0 0"/>
-        </xacro:inertial_box>
-    </link>
-    <joint name="left_knee_outer_joint" type="fixed">
-        <origin xyz="0 0 -${rod_length/2 + motor_thickness/2}" rpy="0.0 ${pi/2} 0.0"/>
-        <parent link="left_knee_motor_link"/>
-        <child link="left_knee_outer_link"/>
-    </joint>
-    <!-- Left Knee - Link -->
-    <link name="left_knee_link">
-        <visual>
-            <origin xyz="0 0 ${knee_rod_height/2}" rpy="0 0 0"/>
-            <geometry>
-                <box size="${knee_rod_length} ${knee_rod_width} ${knee_rod_height}"/>
-            </geometry>
-            <material name="red"/>
-        </visual>
-        <collision>
-            <origin xyz="0 0 ${knee_rod_height/2}" rpy="0 0 0"/>
-            <geometry>
-                <box size="${knee_rod_length} ${knee_rod_width} ${knee_rod_height}"/>
-            </geometry>
-            <material name="red"/>
-        </collision>
-        <xacro:inertial_box mass="${knee_rod_mass}" x="${knee_rod_length}" y="${knee_rod_width}" z="${knee_rod_height}">
-            <origin xyz="0 0 ${knee_rod_height/2}" rpy="0 0 0"/>
-        </xacro:inertial_box>
-    </link>
-    <joint name="left_knee_joint" type="revolute">
-        <origin xyz="0 0 0" rpy="0.0 ${pi/2} -1.047"/>
-        <parent link="left_knee_motor_link"/>
         <child link="left_knee_link"/>
-        <axis xyz="1.0 0.0 0.0"/>
-        <limit lower="${low_limit}" upper="${high_limit}" velocity="${velocity}" effort="${effort}"/>
-    </joint>
-    <!-- Left Wheel -->
-    <link name="left_wheel">
-        <visual>
-            <origin xyz="0 0 0" rpy="0 0 0"/>
-            <geometry>
-                <cylinder radius="${wheel_radius}" length="${wheel_length}"/>
-            </geometry>
-            <material name="black"/>
-        </visual>
-        <collision>
-            <origin xyz="0 0 0" rpy="0 0 0"/>
+        <axis xyz="0.0 -1.0 0.0"/>
+        <limit lower="${low_limit}" upper="${high_limit}" velocity="${velocity}" effort="${effort}"/>
+    </joint>
+    <link name="left_wheel_link">
+        <visual>
+            <origin xyz="0.0 0.0 0.0" rpy="0.0 0.0 0.0"/>
+            <geometry>
+                <cylinder radius="${wheel_radius}" length="${wheel_length}"/>
+            </geometry>
+        </visual>
+        <collision>
+            <origin xyz="0.0 0.0 0.0" rpy="0.0 0.0 0.0"/>
             <geometry>
                 <cylinder radius="${wheel_radius}" length="${wheel_length}"/>
@@ -195,14 +122,14 @@
         </collision>
         <xacro:inertial_cylinder mass="${wheel_mass}" length="${wheel_length}" radius="${wheel_radius}">
-            <origin xyz="0 0 0" rpy="0 0 0"/>
+            <origin xyz="0.0 0.0 0.0" rpy="0.0 0.0 0.0"/>
         </xacro:inertial_cylinder>
     </link>
     <joint name="left_wheel_joint" type="continuous">
-      <origin xyz="${wheel_offset_x} 0 ${wheel_offset_z}" rpy="0 ${pi/2} 0"/>
-      <parent link="left_knee_link"/>
-      <child link="left_wheel"/>
-      <axis xyz="0.0 0.0 1.0"/>
-    </joint>
-    <!-- Right Hip - Gearbox -->
+        <parent link="left_knee_link"/>
+        <child link="left_wheel_link"/>
+        <origin xyz="0 -${rod_length/2 + wheel_length/2} ${rod_height}" rpy="${pi/2} 0.0 0.0"/>
+        <axis xyz="0.0 0.0 1.0"/>
+    </joint>
+        <!-- Right Hip - Gearbox -->
     <link name="right_hip_motor_link">
         <visual>
@@ -225,5 +152,5 @@
     </link>
     <joint name="right_hip_motor_joint" type="revolute">
-        <origin xyz="0.0 -${gearbox_offset_y} 0.0" rpy="${pi/2} -0.524 0.0"/>
+        <origin xyz="0.0 -${gearbox_offset_y} 0.0" rpy="${pi/2} -${pi/6} 0.0"/>
         <parent link="base_link"/>
         <child link="right_hip_motor_link"/>
@@ -231,117 +158,63 @@
         <limit lower="${low_limit}" upper="${high_limit}" velocity="${velocity}" effort="${effort}"/>
     </joint>
-    <!-- Right Hip - Hip -->
     <link name="right_hip_link">
         <visual>
-            <origin xyz="-${rod_height/2} 0 0" rpy="0 ${pi/2} 0"/>
-            <geometry>
-                <box size="${rod_length} ${rod_width} ${rod_height}"/>
-            </geometry>
-            <material name="red"/>
-        </visual>
-        <collision>
-            <origin xyz="-${rod_height/2} 0 0" rpy="0 ${pi/2} 0"/>
-            <geometry>
-                <box size="${rod_length} ${rod_width} ${rod_height}"/>
-            </geometry>
-            <material name="red"/>
-        </collision>
-        <xacro:inertial_box mass="${rod_mass}" x="${rod_length}" y="${rod_width}" z="${rod_height}">
-            <origin xyz="-${rod_height/2} 0 0" rpy="0 ${pi/2} 0"/>
+             <origin xyz="-${rod_height/2} 0 0" rpy="0 ${pi/2} 0"/>
+            <geometry>
+                <box size="${rod_length} ${rod_width} ${rod_height}" rpy="0 0 0"/>
+            </geometry>
+            <material name="red"/>
+        </visual>
+        <collision>
+             <origin xyz="-${rod_height/2} 0 0" rpy="0 ${pi/2} 0"/>
+            <geometry>
+                <box size="${rod_length} ${rod_width} ${rod_height}" rpy="0 0 0"/>
+            </geometry>
+            <material name="red"/>
+        </collision>
+        <xacro:inertial_box mass="${rod_mass}" x="${rod_length}" y="${rod_width}" z="${rod_height}">
+             <origin xyz="-${rod_height/2} 0 0" rpy="0 ${pi/2} 0"/>
         </xacro:inertial_box>
     </link>
     <joint name="right_hip_joint" type="fixed">
-        <origin xyz="0.0 0.0 ${hip_offset_z}" rpy="0.0 0.0 0.0"/>
+        <origin xyz="0.0 0 ${gearbox_thickness/2 + rod_length/2}" rpy="0 0 0"/>
         <parent link="right_hip_motor_link"/>
         <child link="right_hip_link"/>
     </joint>
-    <!-- right Knee - Motor -->
-    <link name="right_knee_motor_link">
-        <visual>
-            <origin xyz="${rod_height} 0 0" rpy="0 0 0"/>
-            <geometry>
-                <cylinder radius="${motor_radius}" length="${motor_thickness}"/>
-            </geometry>
-            <material name="red"/>
-        </visual>
-        <collision>
-            <origin xyz="${rod_height} 0 0" rpy="0 0 0"/>
-            <geometry>
-                <cylinder radius="${motor_radius}" length="${motor_thickness}"/>
-            </geometry>
-            <material name="red"/>
-        </collision>
-        <xacro:inertial_cylinder mass="${motor_mass}" length="${motor_thickness}" radius="${motor_radius}">
-            <origin xyz="${rod_height} 0 0" rpy="0 0 0"/>
-        </xacro:inertial_cylinder>
-    </link>
-    <joint name="right_knee_motor_joint" type="fixed">
-        <origin xyz="${motor_offset_x} 0 ${motor_offset_z}" rpy="0.0 0 0"/>
+    <link name="right_knee_link">
+        <visual>
+             <origin xyz="0 0 ${rod_height/2}" rpy="0.0 0 ${pi/2}"/>
+            <geometry>
+                <box size="${rod_length} ${rod_width} ${rod_height}" rpy="0 0 0"/>
+            </geometry>
+            <material name="red"/>
+        </visual>
+        <collision>
+             <origin xyz="0 0 ${rod_height/2}" rpy="0 0 ${pi/2}"/>
+            <geometry>
+                <box size="${rod_length} ${rod_width} ${rod_height}" rpy="0 0 0"/>
+            </geometry>
+            <material name="red"/>
+        </collision>
+        <xacro:inertial_box mass="${rod_mass}" x="${rod_length}" y="${rod_width}" z="${rod_height}">
+             <origin xyz="0 0 ${rod_height/2}" rpy="0 0 ${pi/2}"/>
+        </xacro:inertial_box>
+    </link>
+    <joint name="right_knee_joint" type="revolute">
+        <origin xyz="-${rod_height} 0 0" rpy="${pi/2} 0 ${pi/6}"/>
         <parent link="right_hip_link"/>
-        <child link="right_knee_motor_link"/>
-    </joint>
-    <!-- Right Hip - Link Outer-->
-    <link name="right_knee_outer_link">
-        <visual>
-            <origin xyz="0 0 ${rod_height/2}" rpy="0 0 0"/>
-            <geometry>
-                <box size="${rod_length} ${rod_width} ${rod_height}"/>
-            </geometry>
-            <material name="red"/>
-        </visual>
-        <collision>
-            <origin xyz="0 0 ${rod_height/2}" rpy="0 0 0"/>
-            <geometry>
-                <box size="${rod_length} ${rod_width} ${rod_height}"/>
-            </geometry>
-            <material name="red"/>
-        </collision>
-        <xacro:inertial_box mass="${rod_mass}" x="${rod_length}" y="${rod_width}" z="${rod_height}">
-            <origin xyz="0 0 ${rod_height/2}" rpy="0 0 0"/>
-        </xacro:inertial_box>
-    </link>
-    <joint name="right_knee_outer_joint" type="fixed">
-        <origin xyz="0 0 ${rod_length/2 + motor_thickness/2}" rpy="0.0 ${pi/2} 0.0"/>
-        <parent link="right_knee_motor_link"/>
-        <child link="right_knee_outer_link"/>
-    </joint>
-    <!-- Right Knee - Link -->
-    <link name="right_knee_link">
-        <visual>
-            <origin xyz="0 0 ${knee_rod_height/2}" rpy="0 0 0"/>
-            <geometry>
-                <box size="${knee_rod_length} ${knee_rod_width} ${knee_rod_height}"/>
-            </geometry>
-            <material name="red"/>
-        </visual>
-        <collision>
-            <origin xyz="0 0 ${knee_rod_height/2}" rpy="0 0 0"/>
-            <geometry>
-                <box size="${knee_rod_length} ${knee_rod_width} ${knee_rod_height}"/>
-            </geometry>
-            <material name="red"/>
-        </collision>
-        <xacro:inertial_box mass="${knee_rod_mass}" x="${knee_rod_length}" y="${knee_rod_width}" z="${knee_rod_height}">
-            <origin xyz="0 0 ${knee_rod_height/2}" rpy="0 0 0"/>
-        </xacro:inertial_box>
-    </link>
-    <joint name="right_knee_joint" type="revolute">
-        <origin xyz="0 0 0" rpy="0.0 ${pi/2} -1.047"/>
-        <parent link="right_knee_motor_link"/>
         <child link="right_knee_link"/>
-        <axis xyz="1.0 0.0 0.0"/>
-        <limit lower="${low_limit}" upper="${high_limit}" velocity="${velocity}" effort="${effort}"/>
-    </joint>
-    <!-- Right Wheel -->
-    <link name="right_wheel">
-        <visual>
-            <origin xyz="0 0 0" rpy="0 0 0"/>
-            <geometry>
-                <cylinder radius="${wheel_radius}" length="${wheel_length}"/>
-            </geometry>
-            <material name="black"/>
-        </visual>
-        <collision>
-            <origin xyz="0 0 0" rpy="0 0 0"/>
+        <axis xyz="0.0 -1.0 0.0"/>
+        <limit lower="${low_limit}" upper="${high_limit}" velocity="${velocity}" effort="${effort}"/>
+    </joint>
+    <link name="right_wheel_link">
+        <visual>
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
Commit message: updated policy and urdf

File: werdna_description/urdf/consts.xacro (robot description, xacro)
@@ -25,6 +25,6 @@
     <xacro:property name="chassis_width" value="0.15"/>
     <xacro:property name="chassis_height" value="0.12"/>
-    <xacro:property name="wheel_radius" value="0.06"/>
-    <xacro:property name="wheel_length" value="0.02"/>
+    <xacro:property name="wheel_radius" value="0.08255"/>
+    <xacro:property name="wheel_length" value="0.045"/>
     <xacro:property name="gearbox_radius" value="0.055"/>
     <xacro:property name="gearbox_thickness" value="0.0738"/>
@@ -38,5 +38,5 @@
     <xacro:property name="chassis_mass" value="2.0"/>
     <xacro:property name="rod_mass" value="0.1"/>
-    <xacro:property name="wheel_mass" value="0.5"/>
+    <xacro:property name="wheel_mass" value="0.65"/>
     <xacro:property name="gearbox_mass" value="0.3"/>
     <xacro:property name="imu_mass" value="0.001"/>
