Commit message: Fixed something

File: werdna_description/ros2_control/ros2_control.xacro (robot description, xacro)
@@ -3,14 +3,5 @@
     <ros2_control name="werdna_ros2_control" type="system">
         <hardware>
-            <plugin>werdna_hardware_interface/WerdnaControlHardware</plugin>
-            <param name="left_hip_name">left_hip_motor_joint</param>
-            <param name="left_knee_name">left_knee_joint</param>
-            <param name="left_wheel_name">left_wheel_joint</param>
-            <param name="right_hip_name">right_hip_motor_joint</param>
-            <param name="right_knee_name">right_knee_joint</param>
-            <param name="right_wheel_name">right_wheel_joint</param>
-            <param name="device">/dev/ttyACM0</param>
-            <param name="baud_rate">115200</param>
-            <param name="timeout_ms">1000</param>
+            <plugin>pi3hat_hardware_interface/Pi3HatControlHardware</plugin>
         </hardware>
         <joint name="left_hip_motor_joint">
@@ -18,4 +9,8 @@
             <state_interface name="position"/>
             <state_interface name="velocity"/>
+            <param name="can_channel">1</param>
+            <param name="can_id">1</param>
+            <param name="position_offset">-0.1</param>
+            <param name="control_mode">position</param>
         </joint>
         <joint name="left_knee_joint">
@@ -23,14 +18,26 @@
             <state_interface name="position"/>
             <state_interface name="velocity"/>
+            <param name="can_channel">1</param>
+            <param name="can_id">2</param>
+            <param name="position_offset">-0.0</param>
+            <param name="control_mode">position</param>
         </joint>
-        <joint name="left_wheel_joint">
+        <!-- <joint name="left_wheel_joint">
             <command_interface name="effort"/>
             <state_interface name="position"/>
             <state_interface name="velocity"/>
-        </joint>
+            <param name="can_channel">1</param>
+            <param name="can_id">3</param>
+            <param name="position_offset">-0.1</param>
+            <param name="control_mode">effort</param>
+        </joint> -->
         <joint name="right_hip_motor_joint">
             <command_interface name="position"/>
             <state_interface name="position"/>
             <state_interface name="velocity"/>
+            <param name="can_channel">2</param>
+            <param name="can_id">4</param>
+            <param name="position_offset">-0.0</param>
+            <param name="control_mode">position</param>
         </joint>
         <joint name="right_knee_joint">
@@ -38,10 +45,18 @@
             <state_interface name="position"/>
             <state_interface name="velocity"/>
+            <param name="can_channel">2</param>
+            <param name="can_id">5</param>
+            <param name="position_offset">-0.0</param>
+            <param name="control_mode">position</param>
         </joint>
-        <joint name="right_wheel_joint">
+        <!-- <joint name="right_wheel_joint">
             <command_interface name="effort"/>
             <state_interface name="position"/>
             <state_interface name="velocity"/>
-        </joint>
+            <param name="can_channel">2</param>
+            <param name="can_id">6</param>
+            <param name="position_offset">-0.0</param>
+            <param name="control_mode">effort</param>
+        </joint> -->
     </ros2_control>
 </robot>

Commit message: RPI

File: werdna_description/ros2_control/ros2_control.xacro (robot description, xacro)
@@ -11,5 +11,5 @@
             <param name="can_channel">1</param>
             <param name="can_id">1</param>
-            <param name="position_offset">-0.1</param>
+            <param name="position_offset">1.5</param>
             <param name="control_mode">position</param>
         </joint>
@@ -20,5 +20,5 @@
             <param name="can_channel">1</param>
             <param name="can_id">2</param>
-            <param name="position_offset">-0.0</param>
+            <param name="position_offset">-0.8</param>
             <param name="control_mode">position</param>
         </joint>
@@ -38,5 +38,5 @@
             <param name="can_channel">2</param>
             <param name="can_id">4</param>
-            <param name="position_offset">-0.0</param>
+            <param name="position_offset">1.5</param>
             <param name="control_mode">position</param>
         </joint>
@@ -47,5 +47,5 @@
             <param name="can_channel">2</param>
             <param name="can_id">5</param>
-            <param name="position_offset">-0.0</param>
+            <param name="position_offset">-0.8</param>
             <param name="control_mode">position</param>
         </joint>

File: werdna_description/urdf/consts.xacro (robot description, xacro)
@@ -43,5 +43,5 @@
     <xacro:property name="chassis_mass" value="1.5"/>
     <xacro:property name="rod_mass" value="0.1"/>
-    <xacro:property name="knee_rod_mass" value="0.2"/>
+    <xacro:property name="knee_rod_mass" value="0.1"/>
     <xacro:property name="wheel_mass" value="0.5"/>
     <xacro:property name="motor_mass" value="0.3"/>

Commit message: Updated Description

File: werdna_description/ros2_control/ros2_control.xacro (robot description, xacro)
@@ -26,5 +26,5 @@
             <param name="control_mode">position</param>
         </joint>
-        <!-- <joint name="left_wheel_joint">
+        <joint name="left_wheel_joint">
             <command_interface name="effort"/>
             <state_interface name="position"/>
@@ -32,7 +32,7 @@
             <param name="can_channel">1</param>
             <param name="can_id">3</param>
-            <param name="position_offset">-0.1</param>
+            <param name="position_offset">0.0</param>
             <param name="control_mode">effort</param>
-        </joint> -->
+        </joint>
         <joint name="right_hip_motor_joint">
             <command_interface name="position"/>

Commit message: Fixed FK on Odom

File: werdna_description/ros2_control/ros2_control.xacro (robot description, xacro)
@@ -53,5 +53,5 @@
             <param name="control_mode">position</param>
         </joint>
-        <!-- <joint name="right_wheel_joint">
+        <joint name="right_wheel_joint">
             <command_interface name="effort"/>
             <state_interface name="position"/>
@@ -61,5 +61,5 @@
             <param name="position_offset">-0.0</param>
             <param name="control_mode">effort</param>
-        </joint> -->
+        </joint>
     <sensor name="imu_sensor">
         <state_interface name="orientation.x"/>

Commit message: making IMU mounting deg angle modular to modify

File: werdna_description/ros2_control/ros2_control.xacro (robot description, xacro)
@@ -4,7 +4,7 @@
         <hardware>
             <plugin>pi3hat_hardware_interface/Pi3HatControlHardware</plugin>
-            <param name="imu_mounting_deg.yaw">0</param>
+            <param name="imu_mounting_deg.roll">-90</param>
             <param name="imu_mounting_deg.pitch">0</param>
-            <param name="imu_mounting_deg.roll">0</param>
+            <param name="imu_mounting_deg.yaw">90</param>
         </hardware>
         <joint name="left_hip_motor_joint">
@@ -15,4 +15,13 @@
             <param name="can_id">1</param>
             <param name="position_offset">0.0</param>
+            <param name="control_mode">position</param>
+        </joint>
+        <joint name="right_hip_motor_joint">
+            <command_interface name="position"/>
+            <state_interface name="position"/>
+            <state_interface name="velocity"/>
+            <param name="can_channel">2</param>
+            <param name="can_id">4</param>
+            <param name="position_offset">0</param>
             <param name="control_mode">position</param>
         </joint>
@@ -26,4 +35,13 @@
             <param name="control_mode">position</param>
         </joint>
+        <joint name="right_knee_joint">
+            <command_interface name="position"/>
+            <state_interface name="position"/>
+            <state_interface name="velocity"/>
+            <param name="can_channel">2</param>
+            <param name="can_id">5</param>
+            <param name="position_offset">0.0</param>
+            <param name="control_mode">position</param>
+        </joint>
         <joint name="left_wheel_joint">
             <command_interface name="effort"/>
@@ -34,22 +52,4 @@
             <param name="position_offset">0.0</param>
             <param name="control_mode">effort</param>
-        </joint>
-        <joint name="right_hip_motor_joint">
-            <command_interface name="position"/>
-            <state_interface name="position"/>
-            <state_interface name="velocity"/>
-            <param name="can_channel">2</param>
-            <param name="can_id">4</param>
-            <param name="position_offset">0</param>
-            <param name="control_mode">position</param>
-        </joint>
-        <joint name="right_knee_joint">
-            <command_interface name="position"/>
-            <state_interface name="position"/>
-            <state_interface name="velocity"/>
-            <param name="can_channel">2</param>
-            <param name="can_id">5</param>
-            <param name="position_offset">0.0</param>
-            <param name="control_mode">position</param>
         </joint>
         <joint name="right_wheel_joint">

Commit message: Remove knee related contents

File: werdna_description/ros2_control/ros2_control.xacro (robot description, xacro)
@@ -28,5 +28,5 @@
             <param name="control_mode">position</param>
         </joint>
-        <joint name="left_knee_joint">
+        <!-- <joint name="left_knee_joint">
             <command_interface name="position"/>
             <state_interface name="position"/>
@@ -47,5 +47,5 @@
             <param name="position_offset">0</param>
             <param name="control_mode">position</param>
-        </joint>
+        </joint> -->
         <joint name="left_wheel_joint">
             <command_interface name="effort"/>

Commit message: Added Slam and Nav2 stuffs

File: werdna_description/ros2_control/ros2_control.xacro (robot description, xacro)
@@ -9,5 +9,5 @@
             <param name="logging">0</param>
         </hardware>
-        <joint name="left_hip_motor_joint">
+        <joint name="left_hip_joint">
             <command_interface name="position"/>
             <state_interface name="position"/>
@@ -20,5 +20,5 @@
             <param name="axis_direction">1</param>
         </joint>
-        <joint name="right_hip_motor_joint">
+        <joint name="right_hip_joint">
             <command_interface name="position"/>
             <state_interface name="position"/>
@@ -31,27 +31,6 @@
             <param name="axis_direction">1</param>
         </joint>
-        <!-- <joint name="left_knee_joint">
-            <command_interface name="position"/>
-            <state_interface name="position"/>
-            <state_interface name="velocity"/>
-            <state_interface name="effort"/>
-            <param name="can_channel">1</param>
-            <param name="can_id">2</param>
-            <param name="position_offset">-0.1</param>
-            <param name="control_mode">position</param>
-        </joint>
-        <joint name="right_knee_joint">
-            <command_interface name="position"/>
-            <state_interface name="position"/>
-            <state_interface name="velocity"/>
-            <state_interface name="effort"/>
-            <param name="can_channel">2</param>
-            <param name="can_id">5</param>
-            <param name="position_offset">0</param>
-            <param name="control_mode">position</param>
-        </joint> -->
         <joint name="left_wheel_joint">
             <command_interface name="effort"/>
-            <!-- <command_interface name="velocity"/>             -->
             <state_interface name="position"/>
             <state_interface name="velocity"/>
@@ -60,10 +39,8 @@
             <param name="can_id">2</param>
             <param name="position_offset">0</param>
-            <!-- <param name="control_mode">velocity</param> -->
             <param name="control_mode">effort</param>
             <param name="axis_direction">-1</param>
         </joint>
         <joint name="right_wheel_joint">
-            <!-- <command_interface name="velocity"/>             -->
             <command_interface name="effort"/>
             <state_interface name="position"/>
@@ -74,5 +51,4 @@
             <param name="position_offset">0</param>
             <param name="control_mode">effort</param>
-            <!-- <param name="control_mode">velocity</param> -->
             <param name="axis_direction">1</param>
         </joint>

File: werdna_description/urdf/consts.xacro (robot description, xacro)
@@ -32,12 +32,17 @@
     <xacro:property name="imu_width" value="0.01"/>
     <xacro:property name="imu_height" value="0.01"/>
+    <xacro:property name="battery_length" value="0.134"/>
+    <xacro:property name="battery_width" value="0.042"/>
+    <xacro:property name="battery_height" value="0.036"/>
     <xacro:property name="rod_length" value="0.008"/>
-    <xacro:property name="rod_width" value="0.02"/>
+    <xacro:property name="rod_width" value="0.05"/>
     <xacro:property name="rod_height" value="0.148"/>
     <!-- Masses -->
-    <xacro:property name="chassis_mass" value="2.0"/>
-    <xacro:property name="rod_mass" value="0.1"/>
-    <xacro:property name="wheel_mass" value="0.65"/>
-    <xacro:property name="gearbox_mass" value="0.3"/>
+    <xacro:property name="chassis_mass" value="1.0"/>
+    <xacro:property name="battery_mass" value="0.5"/>
+    <xacro:property name="knee_rod_mass" value="0.05"/>
+    <xacro:property name="rod_mass" value="0.05"/>
+    <xacro:property name="wheel_mass" value="0.3"/>
+    <xacro:property name="gearbox_mass" value="0.21"/>
     <xacro:property name="imu_mass" value="0.001"/>
     <!-- Offsets -->
@@ -45,9 +50,12 @@
     <xacro:property name="chassis_offset_y" value="0"/>
     <xacro:property name="chassis_offset_z" value="0"/>
+    <xacro:property name="battery_offset_x" value="${chassis_length/2 - battery_width/2}"/>
+    <xacro:property name="battery_offset_y" value="0"/>
+    <xacro:property name="battery_offset_z" value="-${chassis_height/2 + battery_height/2}"/>
     <xacro:property name="imu_offset_x" value="0"/>
     <xacro:property name="imu_offset_y" value="0"/>
     <xacro:property name="imu_offset_z" value="0"/>
     <xacro:property name="gearbox_offset_x" value="0"/>
-    <xacro:property name="gearbox_offset_y" value="${chassis_width/2 + gearbox_thickness/2}"/>
+    <xacro:property name="gearbox_offset_y" value="${chassis_width/2 + rod_length/2}"/>
     <xacro:property name="gearbox_offset_z" value="0"/>
     <xacro:property name="hip_offset_x" value="${-rod_height}"/>

File: werdna_description/urdf/werdna.xacro (robot description, xacro)
@@ -23,4 +23,36 @@
         </collision>
     </link>
+    <link name="battery_link">
+        <xacro:inertial_box mass="${battery_mass}" x="${battery_length}" y="${battery_width}" z="${battery_height}">
+            <origin xyz="0 0 0" rpy="0 0 0"/>
+        </xacro:inertial_box>
+        <visual>
+            <origin xyz="0 0 0" rpy="0.0 0.0 0.0"/>
+            <geometry>
+                <box size="${battery_length} ${battery_width} ${battery_height}"/>
+            </geometry>
+            <material name="blue"/>
+        </visual>
+        <collision>
+            <origin xyz="0 0 0" rpy="0.0 0.0 0.0"/>
+            <geometry>
+                <box size="${battery_length} ${battery_width} ${battery_height}"/>
+            </geometry>
+            <material name="blue"/>
+        </collision>
+    </link>
+    <joint name="battery_joint" type="fixed">
+        <origin xyz="${battery_offset_x} ${battery_offset_y} ${battery_offset_z}" rpy="0.0 0.0 ${pi/2}"/>
+        <parent link="base_link"/>
+        <child link="battery_link"/>
+    </joint>
+    <!-- BASE_FOOTPRINT LINK -->
+    <joint name="base_footprint_joint" type="fixed">
+        <parent link="base_link"/>
+        <child link="base_footprint"/>
+        <origin xyz="0 0 0" rpy="0 0 0"/>
+    </joint>
+    <link name="base_footprint">
+    </link>
     <!-- imu -->
     <!-- <link name="imu_link"></link> -->
@@ -32,5 +64,5 @@
     </joint> -->
     <!-- Left Hip - Gearbox -->
-    <link name="left_hip_motor_link">
+    <!-- <link name="left_hip_motor_link">
         <visual>
             <origin xyz="0 0 0" rpy="0 0 0"/>
@@ -56,6 +88,6 @@
         <child link="left_hip_motor_link"/>
         <axis xyz="0.0 0.0 1.0"/>
-        <limit lower="${low_limit}" upper="${high_limit}" velocity="${velocity}" effort="${effort}"/>
-    </joint>
+        <limit lower="-0.524" upper="0.524" velocity="10" effort="20"/>
+    </joint> -->
     <link name="left_hip_link">
         <visual>
@@ -77,8 +109,10 @@
         </xacro:inertial_box>
     </link>
-    <joint name="left_hip_joint" type="fixed">
-        <origin xyz="0.0 0 -${gearbox_thickness/2 + rod_length/2}" rpy="0 0 0"/>
-        <parent link="left_hip_motor_link"/>
+    <joint name="left_hip_joint" type="revolute">
+        <origin xyz="0.0 ${gearbox_offset_y} 0.0" rpy="${pi/2} -${pi/6} 0.0"/>
+        <parent link="base_link"/>
         <child link="left_hip_link"/>
+        <axis xyz="0.0 0.0 1.0"/>
+        <limit lower="-0.524" upper="0.524" velocity="10" effort="20"/>
     </joint>
     <link name="left_knee_link">
@@ -97,5 +131,5 @@
             <material name="red"/>
         </collision>
-        <xacro:inertial_box mass="${rod_mass}" x="${rod_length}" y="${rod_width}" z="${rod_height}">
+        <xacro:inertial_box mass="${knee_rod_mass}" x="${rod_length}" y="${rod_width}" z="${rod_height}">
              <origin xyz="0 0 ${rod_height/2}" rpy="0 0 ${pi/2}"/>
         </xacro:inertial_box>
@@ -106,5 +140,5 @@
         <child link="left_knee_link"/>
         <axis xyz="0.0 -1.0 0.0"/>
-        <limit lower="${low_limit}" upper="${high_limit}" velocity="${velocity}" effort="${effort}"/>
+        <limit lower="0" upper="1.047" velocity="${velocity}" effort="${effort}"/>
     </joint>
     <link name="left_wheel_link">
@@ -132,5 +166,5 @@
     </joint>
         <!-- Right Hip - Gearbox -->
-    <link name="right_hip_motor_link">
+    <!-- <link name="right_hip_motor_link">
         <visual>
             <origin xyz="0 0 0" rpy="0 0 0"/>
@@ -156,6 +190,6 @@
         <child link="right_hip_motor_link"/>
         <axis xyz="0.0 0.0 1.0"/>
-        <limit lower="${low_limit}" upper="${high_limit}" velocity="${velocity}" effort="${effort}"/>
-    </joint>
+                <limit lower="-0.524" upper="0.524" velocity="10" effort="20"/>
+    </joint> -->
     <link name="right_hip_link">
         <visual>
@@ -177,8 +211,10 @@
         </xacro:inertial_box>
     </link>
-    <joint name="right_hip_joint" type="fixed">
-        <origin xyz="0.0 0 ${gearbox_thickness/2 + rod_length/2}" rpy="0 0 0"/>
-        <parent link="right_hip_motor_link"/>
+    <joint name="right_hip_joint" type="revolute">
+        <origin xyz="0.0 -${gearbox_offset_y} 0.0" rpy="${pi/2} -${pi/6} 0.0"/>
+        <parent link="base_link"/>
         <child link="right_hip_link"/>
+        <axis xyz="0.0 0.0 1.0"/>
+        <limit lower="-0.524" upper="0.524" velocity="10" effort="20"/>
     </joint>
     <link name="right_knee_link">
@@ -197,5 +233,5 @@
             <material name="red"/>
         </collision>
-        <xacro:inertial_box mass="${rod_mass}" x="${rod_length}" y="${rod_width}" z="${rod_height}">
+        <xacro:inertial_box mass="${knee_rod_mass}" x="${rod_length}" y="${rod_width}" z="${rod_height}">
              <origin xyz="0 0 ${rod_height/2}" rpy="0 0 ${pi/2}"/>
         </xacro:inertial_box>
@@ -206,5 +242,5 @@
         <child link="right_knee_link"/>
         <axis xyz="0.0 -1.0 0.0"/>
-        <limit lower="${low_limit}" upper="${high_limit}" velocity="${velocity}" effort="${effort}"/>
+        <limit lower="0" upper="1.047" velocity="${velocity}" effort="${effort}"/>
     </joint>
     <link name="right_wheel_link">
@@ -220,4 +256,11 @@
                 <cylinder radius="${wheel_radius}" length="${wheel_length}"/>
             </geometry>
+             <surface>
+                <contact>
+                <ode>
+                    <mu>0.5</mu>
+                </ode>
+                </contact>
+            </surface>
         </collision>
         <xacro:inertial_cylinder mass="${wheel_mass}" length="${wheel_length}" radius="${wheel_radius}">
